File: PCB/IntegratedOF1.kicad_pcb (KiCad board)
At the start: 2 copper layers, 347 x 156.5 mm, 81 parts, among them J1 USB C Connector, J2 JTAG_TC2030, J3 Conn_01x02_Pin, SW1 Boot, U1 XC6206, U2 USBLC6-2SC6, U3 RP2040, U4 W25Q128JVS, Y1 12MHz

Commit message: Added lite aspects
Parts:
- removed J3: Conn_01x02_Pin, Connector_PinHeader_2.54mm:PinHeader_1x02_P2.54mm_Vertical
- removed MX1, MX11, MX13, MX16, MX18, MX20, MX22, MX24, MX25, MX27, MX3, MX30, MX31, MX34, MX35, MX37, MX40, MX6, MX7, MX9: MX_SW_HS, PCM_marbastlib-mx:SW_MX_HS_1u
- added MX4: MX_SW_solder, MicroGRAM:Kailh_socket_PG1350, F.Cu at (133.7, 39.1)
- added REF**: GRAM_LOGO, MicroGRAM:GRAM_LOGO, F.Cu at (76.2, 158.9)
- MX10, MX12, MX14, MX15, MX17, MX19, MX2, MX21, MX23, MX26, MX28, MX29, MX32, MX33, MX36, MX38, MX39, MX4, MX5, MX8: footprint PCM_marbastlib-mx:SW_MX_1u -> MicroGRAM:Kailh_socket_PG1350
- moved MX15 36.9 mm to (303.9, 38.6)
- moved MX14 36.8 mm to (275.6, 40.4)
- moved MX17 35.2 mm to (332.5, 49.7)
- moved MX12 35.1 mm to (251.4, 56.6)
- moved MX32 32.6 mm to (246.4, 117.1)
- moved MX21 32.1 mm to (280.3, 67.7)
- moved MX23 32.1 mm to (308.7, 65.7)
- moved MX26 30.6 mm to (337.3, 76.9)
- moved MX19 30.3 mm to (256.2, 84.1)
- moved MX33 30.2 mm to (226.7, 136.7)
- moved MX5 29.2 mm to (100.7, 62.8)
- moved MX8 28.7 mm to (129.1, 64.9)
- moved MX4 28.2 mm to (72.9, 74.5)
- moved MX39 27.8 mm to (274.0, 125.3)
- moved MX10 26.3 mm to (153.1, 81.5)
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Connections:
- U3 pad 3: unconnected-(U3-GPIO1-Pad3) -> W
Routing:
- net W: track 0.00 -> 80.3 mm, vias 0 -> 1
- net LEFT: track 181.6 -> 139.5 mm, vias 0 -> 1
- net RIGHT: track 116.8 -> 75.6 mm, vias 0 -> 1
- net DOWN: track 155.6 -> 115.9 mm, vias 0 -> 1
- net L: track 191.0 -> 164.5 mm, vias 0 -> 1
- net M1: track 141.6 -> 117.4 mm, vias 0 -> 1
- net START: track 56.8 -> 34.6 mm
- net C_RT: track 169.2 -> 150.7 mm, vias 0 -> 1
- net Z: track 203.6 -> 220.0 mm, vias 0 -> 1
- net C_DN: track 245.0 -> 230.5 mm, vias 0 -> 1
- net C_UP: track 173.6 -> 187.9 mm, vias 0 -> 1
- net M2: track 155.8 -> 144.3 mm, vias 0 -> 1
- net UP: track 215.3 -> 204.2 mm, vias 0 -> 1
- net C_LT: track 212.8 -> 223.3 mm, vias 0 -> 1
- net X: track 177.3 -> 186.1 mm, vias 0 -> 1
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Other:
- board size 347 x 156.5 mm -> 297.9 x 155 mm
- board text removed: "BOOT"
- board text removed: "Integrated Open Frame 1 made by Quark"
